File: Hardware/PCB/MoonStalker.sch (KiCad schematic (older format))
At the start: 3 parts

Commit message: Added components for DCDC converter and BlueTooth radio
Parts:
- added U3: TEL3-1211, symbol TEL3-1211
- added U4: HC-05_Bluetooth_Radio, symbol HC-05_Bluetooth_Radio
- gave numbers to parts that had none: 3
Connections:
- net at U5.3 (1/TX): now also U4.5 (RXD)
- net VCC: now reaches U5.32 (VIN)
- net VCC: now also U4.2 (VCC)
- net at U5.4 (0/RX): now also U4.4 (TXD)
- new net GND: U4.3 (GND)
Other:
- moved on the sheet: U1, U2, U5
Changed lines of the file:
@@
 LIBS:valves
 LIBS:MoonStalker
+LIBS:MoonStalker-cache
 EELAYER 25 0
 EELAYER END
@@
 encoding utf-8
 Sheet 1 1
-Title ""
-Date ""
-Rev ""
-Comp ""
-Comment1 ""
+Title "MoonStalker Drive Unit"
+Date "2016-01-08"
+Rev "0.1"
+Comp "Koza d.o.o."
+Comment1 "It is very nice"
 Comment2 ""
 Comment3 ""
@@
 $EndDescr
 $Comp
-L Arduino_Micro U?
+L Arduino_Micro U5
 U 1 1 568D949D
-P 5800 3350
-F 0 "U?" H 5800 2400 60  0000 C CNN
-F 1 "Arduino_Micro" H 5800 4400 60  0000 C CNN
-F 2 "" H 5850 3100 60  0000 C CNN
-F 3 "" H 5850 3100 60  0000 C CNN
-	1    5800 3350
+P 7150 4050
+F 0 "U5" H 7150 3100 60  0000 C CNN
+F 1 "Arduino_Micro" H 7150 5100 60  0000 C CNN
+F 2 "" H 7200 3800 60  0000 C CNN
+F 3 "" H 7200 3800 60  0000 C CNN
+	1    7150 4050
 	1    0    0    -1
 $EndComp
 $Comp
-L Pololu_DRV8825 U?
+L Pololu_DRV8825 U1
 U 1 1 568D968D
-P 2600 2850
-F 0 "U?" H 2600 2350 60  0000 C CNN
-F 1 "Pololu_DRV8825" H 2600 3350 60  0000 C CNN
-F 2 "" H 2700 2550 60  0000 C CNN
-F 3 "" H 2700 2550 60  0000 C CNN
-	1    2600 2850
+P 2250 1900
+F 0 "U1" H 2250 1400 60  0000 C CNN
+F 1 "Pololu_DRV8825" H 2250 2400 60  0000 C CNN
+F 2 "" H 2350 1600 60  0000 C CNN
+F 3 "" H 2350 1600 60  0000 C CNN
+	1    2250 1900
 	1    0    0    -1
 $EndComp
 $Comp
-L Pololu_DRV8825 U?
+L Pololu_DRV8825 U2
 U 1 1 568D96DA
-P 2550 5000
-F 0 "U?" H 2550 4500 60  0000 C CNN
-F 1 "Pololu_DRV8825" H 2550 5500 60  0000 C CNN
-F 2 "" H 2650 4700 60  0000 C CNN
-F 3 "" H 2650 4700 60  0000 C CNN
-	1    2550 5000
+P 2250 3600
+F 0 "U2" H 2250 3100 60  0000 C CNN
+F 1 "Pololu_DRV8825" H 2250 4100 60  0000 C CNN
+F 2 "" H 2350 3300 60  0000 C CNN
+F 3 "" H 2350 3300 60  0000 C CNN
+	1    2250 3600
 	1    0    0    -1
 $EndComp
+$Comp
+L HC-05_Bluetooth_Radio U4
+U 1 1 568EE7E0
+P 7150 1350
+F 0 "U4" H 7600 1300 60  0000 C CNN
+F 1 "HC-05_Bluetooth_Radio" H 7200 1700 60  0000 C CNN
+F 2 "" H 7250 1200 60  0000 C CNN
+F 3 "" H 7250 1200 60  0000 C CNN
+	1    7150 1350
+	1    0    0    -1
+$EndComp
+$Comp
+L TEL3-1211 U3
+U 1 1 568EF545
+P 2350 6700
+F 0 "U3" H 2350 6100 60  0000 C CNN
+F 1 "TEL3-1211" H 2350 7250 60  0000 C CNN
+F 2 "" H 1950 6650 60  0000 C CNN
+F 3 "" H 1950 6650 60  0000 C CNN
+	1    2350 6700
+	1    0    0    -1
+$EndComp
+Wire Wire Line
+	7200 1900 7200 2550
+Wire Wire Line
+	7200 2550 6100 2550
+Wire Wire Line
+	6100 2550 6100 3500
+Wire Wire Line
+	6100 3500 6450 3500
+Wire Wire Line
+	7300 1900 7300 2650
+Wire Wire Line
+	7300 2650 6200 2650
+Wire Wire Line
+	6200 2650 6200 3400
+Wire Wire Line
+	6200 3400 6450 3400
+$Comp
+L VCC #PWR01
+U 1 1 568EF868
+P 8300 3400
+F 0 "#PWR01" H 8300 3250 50  0001 C CNN
+F 1 "VCC" H 8300 3550 50  0000 C CNN
+F 2 "" H 8300 3400 50  0000 C CNN
+F 3 "" H 8300 3400 50  0000 C CNN
+	1    8300 3400
+	1    0    0    -1
+$EndComp
+Wire Wire Line
+	8300 3400 7850 3400
+$Comp
+L VCC #PWR02
+U 1 1 568EF93E
+P 6700 2150
+F 0 "#PWR02" H 6700 2000 50  0001 C CNN
+F 1 "VCC" H 6700 2300 50  0000 C CNN
+F 2 "" H 6700 2150 50  0000 C CNN
+F 3 "" H 6700 2150 50  0000 C CNN
+	1    6700 2150
+	1    0    0    -1
+$EndComp
+$Comp
+L GND #PWR03
+U 1 1 568EF95C
+P 7100 2200
+F 0 "#PWR03" H 7100 1950 50  0001 C CNN
+F 1 "GND" H 7100 2050 50  0000 C CNN
+F 2 "" H 7100 2200 50  0000 C CNN
+F 3 "" H 7100 2200 50  0000 C CNN
+	1    7100 2200
+	1    0    0    -1
+$EndComp
+Wire Wire Line
+	7100 1900 7100 2200
+Wire Wire Line
+	6700 2150 7000 2150
+Wire Wire Line
+	7000 2150 7000 1900
 $EndSCHEMATC

Commit message: Added a few more connections to the schematic
Parts:
- added C1: 1000uF, symbol CP
Connections:
- net GND: now also U1.15 (GND), U1.9 (GND), U2.15 (GND), U2.9 (GND), U3.10 (-Vout), U3.15 (-Vout), U5.31 (GND), U5.6 (GND), C1.2
- net VCC: now also U3.11 (+Vout), U3.14 (+Vout), U5.29 (+5V), C1.1; no longer U5.32 (VIN)
- net RXD: now reaches U4.5 (RXD), U5.3 (1/TX)
- net TXD: now reaches U4.4 (TXD), U5.4 (0/RX)
- net at U3.1 (+Vin(VCC)): now also U3.24 (+Vin(VCC))
- net at U3.12 (-Vin(GND)): now also U3.13 (-Vin(GND))
- no-connect marks 0 -> 13
Other:
- moved on the sheet: U3, U4

Commit message: Schematic is now almost complete. An error with DCDC converter power output ports must be fixed and input and output filtering capacitors must be added. Pdf schematic has also been generated.
Parts:
- added C2, C3: 100uF, symbol CP
- added C4: 1000uF, symbol CP
- added P1, P2, P3, P4, P5: CONN_01X02, symbol CONN_01X02
- added R1: 3k3, symbol R
- added R2: 1k, symbol R
Connections:
- net GND: now also U1.1 (~ENABLE), U1.2 (M0), U1.3 (M1), U1.4 (M2), U2.1 (~ENABLE), U2.2 (M0), U2.3 (M1), U2.4 (M2), C2.2, C3.2, C4.2, R2.2
- net VCC: now also U5.30 (RESET), U5.5 (RESET)
- net VERT_STEP: now reaches U5.10 (5(PWM))
- net VERT_STEP: now also U2.7 (STEP)
- net VERT_DIR: now reaches U5.11 (6(PWM)/A7)
- net VERT_DIR: now also U2.8 (DIR)
- net HORIZ_RESET: now reaches U5.12 (7)
- net HORIZ_RESET: now also U1.5 (~RESET)
- net HORIZ_SLEEP: now reaches U5.13 (8/A8)
- net HORIZ_SLEEP: now also U1.6 (~SLEEP)
- net VERT_RESET: now reaches U5.14 (9(PWM)/A9)
- net VERT_RESET: now also U2.5 (~RESET)
- net VERT_SLEEP: now reaches U5.15 (10(PWM)/A10)
- net VERT_SLEEP: now also U2.6 (~SLEEP)
- net HORIZ_FAULT: now reaches U5.16 (11(PWM))
- net HORIZ_FAULT: now also U1.10 (~FAULT)
- net VERT_FAULT: now reaches U5.17 (12/A11)
- net VERT_FAULT: now also U2.10 (~FAULT)
- net VBATT: now reaches U5.21 (A0)
- net VBATT: now also R1.2, R2.1
- net HORIZ_STEP: now reaches U5.7 (2/SDA)
- net HORIZ_STEP: now also U1.7 (STEP)
- net HORIZ_DIR: now reaches U5.8 (3(PWM)/SCL)
- net HORIZ_DIR: now also U1.8 (DIR)
- net at U1.11 (A2): now also P3.2 (P2)
- net at U1.12 (A1): now also P3.1 (P1)
- net at U1.13 (B1): now also P2.2 (P2)
- net at U1.14 (B2): now also P2.1 (P1)
- net VAA: now reaches U1.16 (VMOT)
- net VAA: now also U2.16 (VMOT), U3.1 (+Vin(VCC)), U3.24 (+Vin(VCC)), C2.1, C3.1, C4.1, P1.2 (P2), R1.1
- net at U2.11 (A2): now also P5.2 (P2)
- net at U2.12 (A1): now also P5.1 (P1)
- net at U2.13 (B1): now also P4.2 (P2)
- net at U2.14 (B2): now also P4.1 (P1)
- net at U3.12 (-Vin(GND)), U3.13 (-Vin(GND)): now also P1.1 (P1)
- no-connect marks 13 -> 22
Other:
- note added: "Add DC-DC input and output filtering caps\n"
- note added: "Fix DC-DC power output ERC error"
- note added: "HORIZONTAL DRIVER"
- note added: "TODO:"
- note added: "VERTICAL DRIVER"

Commit message: Fixed some of the power port problems, only one problem remains now.
Connections:
- net GND: now also P1.1 (P1), U3.12 (-Vin(GND)), U3.13 (-Vin(GND))
Changed lines of the file:
@@
 	6050 3500 6450 3500
-Wire Wire Line
-	2950 6450 3050 6450
-Wire Wire Line
-	3050 6450 3050 6750
-Wire Wire Line
-	3050 6750 1550 6750
-Wire Wire Line
-	1550 6750 1550 6450
 Wire Wire Line
 	2950 5400 2950 5650
@@
 Connection ~ 1550 5400
 Wire Wire Line
-	950  5500 1150 5500
-Wire Wire Line
-	1150 5500 1150 6550
-Wire Wire Line
-	1150 6550 1550 6550
-Connection ~ 1550 6550
+	950  5500 1250 5500
 $Comp
 L R R1
@@
 Connection ~ 3050 3350
 NoConn ~ 6450 3300
-$Comp
-L PWR_FLAG #FLG022
-U 1 1 5693173F
-P 1000 5250
-F 0 "#FLG022" H 1000 5345 50  0001 C CNN
-F 1 "PWR_FLAG" H 1000 5430 50  0000 C CNN
-F 2 "" H 1000 5250 50  0000 C CNN
-F 3 "" H 1000 5250 50  0000 C CNN
-	1    1000 5250
-	1    0    0    -1
-$EndComp
-$Comp
-L PWR_FLAG #FLG023
-U 1 1 56931773
-P 950 5850
-F 0 "#FLG023" H 950 5945 50  0001 C CNN
-F 1 "PWR_FLAG" H 950 6030 50  0000 C CNN
-F 2 "" H 950 5850 50  0000 C CNN
-F 3 "" H 950 5850 50  0000 C CNN
-	1    950  5850
-	-1   0    0    1
-$EndComp
-Wire Wire Line
-	950  5850 950  5500
-Wire Wire Line
-	1000 5250 1000 5400
-Connection ~ 1000 5400
 Text Notes 5200 5900 2    79   ~ 0
 TODO:
@@
 Text Notes 6950 6200 2    79   ~ 0
 Fix DC-DC power output ERC error
+$Comp
+L GND #PWR022
+U 1 1 5692E8AB
+P 1550 6550
+F 0 "#PWR022" H 1550 6300 50  0001 C CNN
+F 1 "GND" H 1550 6400 50  0000 C CNN
+F 2 "" H 1550 6550 50  0000 C CNN
+F 3 "" H 1550 6550 50  0000 C CNN
+	1    1550 6550
+	1    0    0    -1
+$EndComp
+$Comp
+L GND #PWR023
+U 1 1 5692E8DF
+P 2950 6550
+F 0 "#PWR023" H 2950 6300 50  0001 C CNN
+F 1 "GND" H 2950 6400 50  0000 C CNN
+F 2 "" H 2950 6550 50  0000 C CNN
+F 3 "" H 2950 6550 50  0000 C CNN
+	1    2950 6550
+	1    0    0    -1
+$EndComp
+Wire Wire Line
+	1550 6450 1550 6550
+Wire Wire Line
+	2950 6450 2950 6550
+Wire Wire Line
+	1250 5500 1250 6250
+$Comp
+L PWR_FLAG #FLG024
+U 1 1 5692ED49
+P 1150 5200
+F 0 "#FLG024" H 1150 5295 50  0001 C CNN
+F 1 "PWR_FLAG" H 1150 5380 50  0000 C CNN
+F 2 "" H 1150 5200 50  0000 C CNN
+F 3 "" H 1150 5200 50  0000 C CNN
+	1    1150 5200
+	1    0    0    -1
+$EndComp
+Wire Wire Line
+	1150 5200 1150 5400
+Connection ~ 1150 5400
 $EndSCHEMATC

Commit message: Added a few decoupling caps to schematic
Parts:
- added C1, C10, C4, C5, C6, C9: 100nF, symbol C
- renumbered C4 to C7, C1 to C8, U5 to U4, U4 to U5
Connections:
- net GND: now also C1.2, C10.2, C4.2, C5.2, C6.2, C9.2
- net VAA: now also C1.1, C4.1, C5.1
- net VCC: now also C10.1, C6.1, C9.1
Other:
- moved on the sheet: C2, C3, C8
