File: Hardware/PCB/MoonStalker.sch (KiCad schematic (older format))
At the start: 22 parts, among them P1 CONN_01X02, P2 CONN_01X02, P3 CONN_01X02, P4 CONN_01X02, P5 CONN_01X02, U1 Pololu_DRV8825, U2 Pololu_DRV8825, U3 TEL3-1211, U4 Arduino_Micro, U5 HC-05_Bluetooth_Radio

Commit message: Fixed TEL3-1211 footprint and removed old text from schematic.
Other:
- note removed: "Add DC-DC input and output filtering caps\n"
- note removed: "Fix DC-DC power output ERC error"
- note removed: "TODO:"
Changed lines of the file:
@@
 Connection ~ 2950 3350
 NoConn ~ 6450 3300
-Text Notes 5200 5900 2    79   ~ 0
-TODO:
-Text Notes 7450 6050 2    79   ~ 0
-Add DC-DC input and output filtering caps\n
-Text Notes 6950 6200 2    79   ~ 0
-Fix DC-DC power output ERC error
 $Comp
 L GND #PWR022

Commit message: Generated netlist and started associating symbols to footprints.
Parts:
- U3: footprint (none) -> MoonStalker:TEL3-1211
Changed lines of the file:
@@
 F 0 "U4" H 7150 3100 60  0000 C CNN
 F 1 "Arduino_Micro" H 7150 5100 60  0000 C CNN
-F 2 "" H 7200 3800 60  0000 C CNN
+F 2 "" H 7200 3800 60  0001 C CNN
 F 3 "" H 7200 3800 60  0000 C CNN
 	1    7150 4050
@@
 F 0 "U1" H 2250 1400 60  0000 C CNN
 F 1 "Pololu_DRV8825" H 2250 2400 60  0000 C CNN
-F 2 "" H 2350 1600 60  0000 C CNN
+F 2 "" H 2350 1600 60  0001 C CNN
 F 3 "" H 2350 1600 60  0000 C CNN
 	1    2250 1900
@@
 F 0 "U2" H 2250 3100 60  0000 C CNN
 F 1 "Pololu_DRV8825" H 2250 4100 60  0000 C CNN
-F 2 "" H 2350 3300 60  0000 C CNN
+F 2 "" H 2350 3300 60  0001 C CNN
 F 3 "" H 2350 3300 60  0000 C CNN
 	1    2250 3600
@@
 F 0 "U5" V 8850 1350 60  0000 C CNN
 F 1 "HC-05_Bluetooth_Radio" V 8000 1450 60  0000 C CNN
-F 2 "" H 8500 1250 60  0000 C CNN
+F 2 "" H 8500 1250 60  0001 C CNN
 F 3 "" H 8500 1250 60  0000 C CNN
 	1    8400 1400
@@
 F 0 "U3" H 2250 5450 60  0000 C CNN
 F 1 "TEL3-1211" H 2250 6600 60  0000 C CNN
-F 2 "" H 1850 6000 60  0000 C CNN
+F 2 "MoonStalker:TEL3-1211" H 1850 6000 60  0001 C CNN
 F 3 "" H 1850 6000 60  0000 C CNN
 	1    2250 6050
@@
 F 0 "C8" H 3925 6850 50  0000 L CNN
 F 1 "1000uF" H 3925 6650 50  0000 L CNN
-F 2 "" H 3938 6600 50  0000 C CNN
+F 2 "" H 3938 6600 50  0001 C CNN
 F 3 "" H 3900 6750 50  0000 C CNN
 	1    3900 6750
@@
 F 0 "P3" H 3900 2500 50  0000 C CNN
 F 1 "CONN_01X02" V 4000 2350 50  0000 C CNN
-F 2 "" H 3900 2350 50  0000 C CNN
+F 2 "" H 3900 2350 50  0001 C CNN
 F 3 "" H 3900 2350 50  0000 C CNN
 	1    3900 2350
@@
 F 0 "P2" H 3900 1950 50  0000 C CNN
 F 1 "CONN_01X02" V 4000 1800 50  0000 C CNN
-F 2 "" H 3900 1800 50  0000 C CNN
+F 2 "" H 3900 1800 50  0001 C CNN
 F 3 "" H 3900 1800 50  0000 C CNN
 	1    3900 1800
@@
 F 0 "P5" H 3950 4200 50  0000 C CNN
 F 1 "CONN_01X02" V 4050 4050 50  0000 C CNN
-F 2 "" H 3950 4050 50  0000 C CNN
+F 2 "" H 3950 4050 50  0001 C CNN
 F 3 "" H 3950 4050 50  0000 C CNN
 	1    3950 4050
@@
 F 0 "P4" H 3950 3650 50  0000 C CNN
 F 1 "CONN_01X02" V 4050 3500 50  0000 C CNN
-F 2 "" H 3950 3500 50  0000 C CNN
+F 2 "" H 3950 3500 50  0001 C CNN
 F 3 "" H 3950 3500 50  0000 C CNN
 	1    3950 3500
@@
 F 0 "P1" H 750 5600 50  0000 C CNN
 F 1 "CONN_01X02" V 850 5450 50  0000 C CNN
-F 2 "" H 750 5450 50  0000 C CNN
+F 2 "" H 750 5450 50  0001 C CNN
 F 3 "" H 750 5450 50  0000 C CNN
 	1    750  5450
@@
 F 0 "R1" V 3980 5550 50  0000 C CNN
 F 1 "3k3" V 3900 5550 50  0000 C CNN
-F 2 "" V 3830 5550 50  0000 C CNN
+F 2 "" V 3830 5550 50  0001 C CNN
 F 3 "" H 3900 5550 50  0000 C CNN
 	1    3900 5550
@@
 F 0 "R2" V 3980 5900 50  0000 C CNN
 F 1 "1k" V 3900 5900 50  0000 C CNN
-F 2 "" V 3830 5900 50  0000 C CNN
+F 2 "" V 3830 5900 50  0001 C CNN
 F 3 "" H 3900 5900 50  0000 C CNN
 	1    3900 5900
@@
 F 0 "C7" H 3625 5750 50  0000 L CNN
 F 1 "1000uF" H 3625 5550 50  0000 L CNN
-F 2 "" H 3638 5500 50  0000 C CNN
+F 2 "" H 3638 5500 50  0001 C CNN
 F 3 "" H 3600 5650 50  0000 C CNN
 	1    3600 5650
@@
 F 0 "C2" H 2900 1650 50  0000 L CNN
 F 1 "100uF" H 2975 1300 50  0000 L CNN
-F 2 "" H 2988 1250 50  0000 C CNN
+F 2 "" H 2988 1250 50  0001 C CNN
 F 3 "" H 2950 1400 50  0000 C CNN
 	1    2950 1400
@@
 F 0 "C3" H 2975 3200 50  0000 L CNN
 F 1 "100uF" H 2975 3000 50  0000 L CNN
-F 2 "" H 2988 2950 50  0000 C CNN
+F 2 "" H 2988 2950 50  0001 C CNN
 F 3 "" H 2950 3100 50  0000 C CNN
 	1    2950 3100
@@
 F 0 "C6" H 3525 6850 50  0000 L CNN
 F 1 "100nF" H 3525 6650 50  0000 L CNN
-F 2 "" H 3538 6600 50  0000 C CNN
+F 2 "" H 3538 6600 50  0001 C CNN
 F 3 "" H 3500 6750 50  0000 C CNN
 	1    3500 6750
@@
 F 0 "C1" H 1275 5700 50  0000 L CNN
 F 1 "100nF" H 1275 5500 50  0000 L CNN
-F 2 "" H 1288 5450 50  0000 C CNN
+F 2 "" H 1288 5450 50  0001 C CNN
 F 3 "" H 1250 5600 50  0000 C CNN
 	1    1250 5600
@@
 F 0 "C9" H 7225 1550 50  0000 L CNN
 F 1 "100nF" H 7225 1350 50  0000 L CNN
-F 2 "" H 7238 1300 50  0000 C CNN
+F 2 "" H 7238 1300 50  0001 C CNN
 F 3 "" H 7200 1450 50  0000 C CNN
 	1    7200 1450
@@
 F 0 "C4" H 3325 1550 50  0000 L CNN
 F 1 "100nF" H 3325 1350 50  0000 L CNN
-F 2 "" H 3338 1300 50  0000 C CNN
+F 2 "" H 3338 1300 50  0001 C CNN
 F 3 "" H 3300 1450 50  0000 C CNN
 	1    3300 1450
@@
 F 0 "C5" H 3325 3250 50  0000 L CNN
 F 1 "100nF" H 3325 3050 50  0000 L CNN
-F 2 "" H 3338 3000 50  0000 C CNN
+F 2 "" H 3338 3000 50  0001 C CNN
 F 3 "" H 3300 3150 50  0000 C CNN
 	1    3300 3150
@@
 F 0 "C10" H 8275 4000 50  0000 L CNN
 F 1 "100nF" H 8275 3800 50  0000 L CNN
-F 2 "" H 8288 3750 50  0000 C CNN
+F 2 "" H 8288 3750 50  0001 C CNN
 F 3 "" H 8250 3900 50  0000 C CNN
 	1    8250 3900

Commit message: Added footprints for Arduino Micro and Pololu DRV8825.
Parts:
- P1, P2, P3, P4, P5: footprint (none) -> Terminal_Blocks:TerminalBlock_Pheonix_MPT-2.54mm_2pol
- R1, R2: footprint (none) -> Resistors_ThroughHole:Resistor_Horizontal_RM7mm
- U1, U2: footprint (none) -> MoonStalker:Pololu_DRV8825
- U4: footprint (none) -> MoonStalker:Arduino_Micro
- U5: footprint (none) -> Socket_Strips:Socket_Strip_Straight_1x06
Changed lines of the file:
@@
 F 0 "U4" H 7150 3100 60  0000 C CNN
 F 1 "Arduino_Micro" H 7150 5100 60  0000 C CNN
-F 2 "" H 7200 3800 60  0001 C CNN
+F 2 "MoonStalker:Arduino_Micro" H 7200 3800 60  0001 C CNN
 F 3 "" H 7200 3800 60  0000 C CNN
 	1    7150 4050
@@
 F 0 "U1" H 2250 1400 60  0000 C CNN
 F 1 "Pololu_DRV8825" H 2250 2400 60  0000 C CNN
-F 2 "" H 2350 1600 60  0001 C CNN
+F 2 "MoonStalker:Pololu_DRV8825" H 2350 1600 60  0001 C CNN
 F 3 "" H 2350 1600 60  0000 C CNN
 	1    2250 1900
@@
 F 0 "U2" H 2250 3100 60  0000 C CNN
 F 1 "Pololu_DRV8825" H 2250 4100 60  0000 C CNN
-F 2 "" H 2350 3300 60  0001 C CNN
+F 2 "MoonStalker:Pololu_DRV8825" H 2350 3300 60  0001 C CNN
 F 3 "" H 2350 3300 60  0000 C CNN
 	1    2250 3600
@@
 F 0 "U5" V 8850 1350 60  0000 C CNN
 F 1 "HC-05_Bluetooth_Radio" V 8000 1450 60  0000 C CNN
-F 2 "" H 8500 1250 60  0001 C CNN
+F 2 "Socket_Strips:Socket_Strip_Straight_1x06" H 8500 1250 60  0001 C CNN
 F 3 "" H 8500 1250 60  0000 C CNN
 	1    8400 1400
@@
 F 0 "P3" H 3900 2500 50  0000 C CNN
 F 1 "CONN_01X02" V 4000 2350 50  0000 C CNN
-F 2 "" H 3900 2350 50  0001 C CNN
+F 2 "Terminal_Blocks:TerminalBlock_Pheonix_MPT-2.54mm_2pol" H 3900 2350 50  0001 C CNN
 F 3 "" H 3900 2350 50  0000 C CNN
 	1    3900 2350
@@
 F 0 "P2" H 3900 1950 50  0000 C CNN
 F 1 "CONN_01X02" V 4000 1800 50  0000 C CNN
-F 2 "" H 3900 1800 50  0001 C CNN
+F 2 "Terminal_Blocks:TerminalBlock_Pheonix_MPT-2.54mm_2pol" H 3900 1800 50  0001 C CNN
 F 3 "" H 3900 1800 50  0000 C CNN
 	1    3900 1800
@@
 F 0 "P5" H 3950 4200 50  0000 C CNN
 F 1 "CONN_01X02" V 4050 4050 50  0000 C CNN
-F 2 "" H 3950 4050 50  0001 C CNN
+F 2 "Terminal_Blocks:TerminalBlock_Pheonix_MPT-2.54mm_2pol" H 3950 4050 50  0001 C CNN
 F 3 "" H 3950 4050 50  0000 C CNN
 	1    3950 4050
@@
 F 0 "P4" H 3950 3650 50  0000 C CNN
 F 1 "CONN_01X02" V 4050 3500 50  0000 C CNN
-F 2 "" H 3950 3500 50  0001 C CNN
+F 2 "Terminal_Blocks:TerminalBlock_Pheonix_MPT-2.54mm_2pol" H 3950 3500 50  0001 C CNN
 F 3 "" H 3950 3500 50  0000 C CNN
 	1    3950 3500
@@
 F 0 "P1" H 750 5600 50  0000 C CNN
 F 1 "CONN_01X02" V 850 5450 50  0000 C CNN
-F 2 "" H 750 5450 50  0001 C CNN
+F 2 "Terminal_Blocks:TerminalBlock_Pheonix_MPT-2.54mm_2pol" H 750 5450 50  0001 C CNN
 F 3 "" H 750 5450 50  0000 C CNN
 	1    750  5450
@@
 F 0 "R1" V 3980 5550 50  0000 C CNN
 F 1 "3k3" V 3900 5550 50  0000 C CNN
-F 2 "" V 3830 5550 50  0001 C CNN
+F 2 "Resistors_ThroughHole:Resistor_Horizontal_RM7mm" V 3830 5550 50  0001 C CNN
 F 3 "" H 3900 5550 50  0000 C CNN
 	1    3900 5550
@@
 F 0 "R2" V 3980 5900 50  0000 C CNN
 F 1 "1k" V 3900 5900 50  0000 C CNN
-F 2 "" V 3830 5900 50  0001 C CNN
+F 2 "Resistors_ThroughHole:Resistor_Horizontal_RM7mm" V 3830 5900 50  0001 C CNN
 F 3 "" H 3900 5900 50  0000 C CNN
 	1    3900 5900

Commit message: Finished schematic, footprints and cvpcb associations. Netlist complete and ready for PCB layout.
Parts:
- C1, C10, C6: value 100nF -> 47nF; footprint (none) -> Capacitors_ThroughHole:C_Rect_L13_W4_P10
- C2, C3: value 100uF -> 220uF; footprint (none) -> Capacitors_ThroughHole:C_Radial_D10_L13_P5
- C4, C5: footprint (none) -> Capacitors_ThroughHole:C_Rect_L7_W2.5_P5
- C7, C8: footprint (none) -> Capacitors_ThroughHole:C_Radial_D10_L16_P5
- C9: value 100nF -> 47nF; footprint (none) -> Capacitors_ThroughHole:C_Rect_L10_W2.5_P7.5
Changed lines of the file:
@@
 F 0 "C8" H 3925 6850 50  0000 L CNN
 F 1 "1000uF" H 3925 6650 50  0000 L CNN
-F 2 "" H 3938 6600 50  0001 C CNN
+F 2 "Capacitors_ThroughHole:C_Radial_D10_L16_P5" H 3938 6600 50  0001 C CNN
 F 3 "" H 3900 6750 50  0000 C CNN
 	1    3900 6750
@@
 F 0 "C7" H 3625 5750 50  0000 L CNN
 F 1 "1000uF" H 3625 5550 50  0000 L CNN
-F 2 "" H 3638 5500 50  0001 C CNN
+F 2 "Capacitors_ThroughHole:C_Radial_D10_L16_P5" H 3638 5500 50  0001 C CNN
 F 3 "" H 3600 5650 50  0000 C CNN
 	1    3600 5650
@@
 P 2950 1400
 F 0 "C2" H 2900 1650 50  0000 L CNN
-F 1 "100uF" H 2975 1300 50  0000 L CNN
-F 2 "" H 2988 1250 50  0001 C CNN
+F 1 "220uF" H 2975 1300 50  0000 L CNN
+F 2 "Capacitors_ThroughHole:C_Radial_D10_L13_P5" H 2988 1250 50  0001 C CNN
 F 3 "" H 2950 1400 50  0000 C CNN
 	1    2950 1400
@@
 P 2950 3100
 F 0 "C3" H 2975 3200 50  0000 L CNN
-F 1 "100uF" H 2975 3000 50  0000 L CNN
-F 2 "" H 2988 2950 50  0001 C CNN
+F 1 "220uF" H 2975 3000 50  0000 L CNN
+F 2 "Capacitors_ThroughHole:C_Radial_D10_L13_P5" H 2988 2950 50  0001 C CNN
 F 3 "" H 2950 3100 50  0000 C CNN
 	1    2950 3100
@@
 P 3500 6750
 F 0 "C6" H 3525 6850 50  0000 L CNN
-F 1 "100nF" H 3525 6650 50  0000 L CNN
-F 2 "" H 3538 6600 50  0001 C CNN
+F 1 "47nF" H 3525 6650 50  0000 L CNN
+F 2 "Capacitors_ThroughHole:C_Rect_L13_W4_P10" H 3538 6600 50  0001 C CNN
 F 3 "" H 3500 6750 50  0000 C CNN
 	1    3500 6750
@@
 P 1250 5600
 F 0 "C1" H 1275 5700 50  0000 L CNN
-F 1 "100nF" H 1275 5500 50  0000 L CNN
-F 2 "" H 1288 5450 50  0001 C CNN
+F 1 "47nF" H 1275 5500 50  0000 L CNN
+F 2 "Capacitors_ThroughHole:C_Rect_L13_W4_P10" H 1288 5450 50  0001 C CNN
 F 3 "" H 1250 5600 50  0000 C CNN
 	1    1250 5600
@@
 P 7200 1450
 F 0 "C9" H 7225 1550 50  0000 L CNN
-F 1 "100nF" H 7225 1350 50  0000 L CNN
-F 2 "" H 7238 1300 50  0001 C CNN
+F 1 "47nF" H 7000 1350 50  0000 L CNN
+F 2 "Capacitors_ThroughHole:C_Rect_L10_W2.5_P7.5" H 7238 1300 50  0001 C CNN
 F 3 "" H 7200 1450 50  0000 C CNN
 	1    7200 1450
@@
 F 0 "C4" H 3325 1550 50  0000 L CNN
 F 1 "100nF" H 3325 1350 50  0000 L CNN
-F 2 "" H 3338 1300 50  0001 C CNN
+F 2 "Capacitors_ThroughHole:C_Rect_L7_W2.5_P5" H 3338 1300 50  0001 C CNN
 F 3 "" H 3300 1450 50  0000 C CNN
 	1    3300 1450
@@
 F 0 "C5" H 3325 3250 50  0000 L CNN
 F 1 "100nF" H 3325 3050 50  0000 L CNN
-F 2 "" H 3338 3000 50  0001 C CNN
+F 2 "Capacitors_ThroughHole:C_Rect_L7_W2.5_P5" H 3338 3000 50  0001 C CNN
 F 3 "" H 3300 3150 50  0000 C CNN
 	1    3300 3150
@@
 P 8250 3900
 F 0 "C10" H 8275 4000 50  0000 L CNN
-F 1 "100nF" H 8275 3800 50  0000 L CNN
-F 2 "" H 8288 3750 50  0001 C CNN
+F 1 "47nF" H 8275 3800 50  0000 L CNN
+F 2 "Capacitors_ThroughHole:C_Rect_L13_W4_P10" H 8288 3750 50  0001 C CNN
 F 3 "" H 8250 3900 50  0000 C CNN
 	1    8250 3900

Commit message: Updated R1 and R2 resistor values to real measured values.
Parts:
- R1: value 3k3 -> 14k93
- R2: value 1k -> 5088R
Changed lines of the file:
@@
 LIBS:atmel
 LIBS:contrib
+LIBS:MoonStalker
 LIBS:valves
-LIBS:MoonStalker
 LIBS:MoonStalker-cache
 EELAYER 25 0
@@
 P 3900 5550
 F 0 "R1" V 3980 5550 50  0000 C CNN
-F 1 "3k3" V 3900 5550 50  0000 C CNN
+F 1 "14k93" V 4050 5550 50  0000 C CNN
 F 2 "Resistors_ThroughHole:Resistor_Horizontal_RM7mm" V 3830 5550 50  0001 C CNN
 F 3 "" H 3900 5550 50  0000 C CNN
@@
 P 3900 5900
 F 0 "R2" V 3980 5900 50  0000 C CNN
-F 1 "1k" V 3900 5900 50  0000 C CNN
+F 1 "5088R" V 4050 5900 50  0000 C CNN
 F 2 "Resistors_ThroughHole:Resistor_Horizontal_RM7mm" V 3830 5900 50  0001 C CNN
 F 3 "" H 3900 5900 50  0000 C CNN
