File: Hardware/PCB/MoonStalker.kicad_pcb (KiCad board)
At the start: 2 copper layers, 91.4 x 86.4 mm, 22 parts, among them P1 CONN_01X02, P2 CONN_01X02, P3 CONN_01X02, P4 CONN_01X02, P5 CONN_01X02, U1 Pololu_DRV8825, U2 Pololu_DRV8825, U3 TEL3-1211, U4 Arduino_Micro, U5 HC-05_Bluetooth_Radio

Commit message: Finished all connections in the pcb layout. Still have to check all DRC rules, add OSHPark limits, make some tracks thicker.
Parts:
- moved P4 10.0 mm to (62.2, 87.0)
- moved P5 9.66 mm to (62.2, 96.5)
Routing:
- net HORIZ_FAULT: track 0.00 -> 71.7 mm, vias 0 -> 2
- net VERT_FAULT: track 0.00 -> 45.4 mm, vias 0 -> 2
- net HORIZ_SLEEP: track 0.00 -> 34.2 mm, vias 0 -> 2
- net HORIZ_RESET: track 0.00 -> 33.8 mm
- net VERT_STEP: track 0.00 -> 32.1 mm, vias 0 -> 2
- net Net-(P5-Pad2): track 0.00 -> 28.9 mm
- net VERT_DIR: track 0.00 -> 28.0 mm, vias 0 -> 2
- net Net-(P5-Pad1): track 0.00 -> 25.7 mm
- net HORIZ_STEP: track 0.00 -> 25.3 mm
- net HORIZ_DIR: track 0.00 -> 20.8 mm
- net Net-(P4-Pad2): track 0.00 -> 20.7 mm
- net Net-(P2-Pad2): track 0.00 -> 18.1 mm
- net Net-(P4-Pad1): track 0.00 -> 17.5 mm
- net Net-(P2-Pad1): track 0.00 -> 15.6 mm
- net VERT_SLEEP: track 29.5 -> 30.3 mm
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
Commit message: Adjusted all track widths and design rules for Osh Park. Mounting holes still missing.
Parts:
- moved C7 17.3 mm to (83.9, 131.9)
- moved C8 7.84 mm to (96.1, 131.9)
Routing:
- net VAA: track 238.0 -> 224.1 mm
- net Net-(P2-Pad2): track 18.1 -> 20.7 mm
- net Net-(P3-Pad2): track 27.0 -> 29.4 mm
- net Net-(P2-Pad1): track 15.6 -> 17.2 mm
- net Net-(P3-Pad1): track 23.3 -> 24.8 mm
- net Net-(P5-Pad1): track 25.7 -> 24.6 mm
- net VERT_STEP: track 32.1 -> 31.5 mm
Other:
- net class Default: clearance 0.2 -> 0.1524; trace_width 0.25 -> 0.4; via_drill 0.4 -> 0.3302
- net class Stepper_traces added: clearance 0.1524, trace_width 0.8, via_dia 0.6, via_drill 0.3302
- rule trace_clearance: 0.2 -> 0.1524
- rule trace_min: 0.2 -> 0.1524
- rule via_min_drill: 0.3 -> 0.3302

Commit message: Added mounting holes and silkscreen logo to the PCB.
Parts:
- added REF**: MountingHole_3.2mm_M3_ISO14580_Pad, Mounting_Holes:MountingHole_3.2mm_M3_ISO14580_Pad, F.Cu at (60.0, 57.5)
- added REF**: MountingHole_3.2mm_M3_ISO14580_Pad, Mounting_Holes:MountingHole_3.2mm_M3_ISO14580_Pad, F.Cu at (140.0, 57.5)
- added REF**: MountingHole_3.2mm_M3_ISO14580_Pad, Mounting_Holes:MountingHole_3.2mm_M3_ISO14580_Pad, F.Cu at (60.0, 132.5)
- added REF**: MountingHole_3.2mm_M3_ISO14580_Pad, Mounting_Holes:MountingHole_3.2mm_M3_ISO14580_Pad, F.Cu at (140.0, 132.5)
Other:
- board text added: "MoonStalker"
- board text added: "V1.0"
Changed lines of the file:
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@@
-(kicad_pcb (version 4) (host pcbnew 4.0.5-e0-6337~49~ubuntu16.04.1)
+(kicad_pcb (version 4) (host pcbnew 4.0.6-e0-6349~53~ubuntu16.04.1)
   (general
     (links 72)
     (no_connects 0)
-    (area 54.534999 53.264999 146.125001 139.775001)
+    (area 44.704743 52.8226 155.295258 139.775001)
     (thickness 1.6)
-    (drawings 4)
+    (drawings 6)
     (tracks 168)
     (zones 0)
-    (modules 22)
+    (modules 26)
     (nets 47)
   )
@@
     (mod_text_size 1 1)
     (mod_text_width 0.15)
-    (pad_size 1.524 1.524)
-    (pad_drill 0.762)
+    (pad_size 5.5 5.5)
+    (pad_drill 3.2)
     (pad_to_mask_clearance 0.2)
     (aux_axis_origin 0 0)
@@
       (outputformat 1)
       (mirror false)
-      (drillshape 1)
+      (drillshape 0)
       (scaleselection 1)
-      (outputdirectory ""))
+      (outputdirectory gerbers/))
   )
   (net 0 "")
@@
     )
   )
+  (module Mounting_Holes:MountingHole_3.2mm_M3_ISO14580_Pad (layer F.Cu)
+    (at 60 57.5)
+    (descr "Mounting Hole 3.2mm, M3, ISO14580")
+    (tags "mounting hole 3.2mm m3 iso14580")
+    (fp_text reference REF** (at 0 -3.75) (layer F.SilkS)
+      (effects (font (size 1 1) (thickness 0.15)))
+    )
+    (fp_text value MountingHole_3.2mm_M3_ISO14580_Pad (at 0 3.75) (layer F.Fab)
+      (effects (font (size 1 1) (thickness 0.15)))
+    )
+    (fp_circle (center 0 0) (end 2.75 0) (layer Cmts.User) (width 0.15))
+    (fp_circle (center 0 0) (end 3 0) (layer F.CrtYd) (width 0.05))
+    (pad 1 thru_hole circle (at 0 0) (size 5.5 5.5) (drill 3.2) (layers *.Cu *.Mask))
+  )
+  (module Mounting_Holes:MountingHole_3.2mm_M3_ISO14580_Pad (layer F.Cu)
+    (at 140 57.5)
+    (descr "Mounting Hole 3.2mm, M3, ISO14580")
+    (tags "mounting hole 3.2mm m3 iso14580")
+    (fp_text reference REF** (at 0 -3.75) (layer F.SilkS)
+      (effects (font (size 1 1) (thickness 0.15)))
+    )
+    (fp_text value MountingHole_3.2mm_M3_ISO14580_Pad (at 0 3.75) (layer F.Fab)
+      (effects (font (size 1 1) (thickness 0.15)))
+    )
+    (fp_circle (center 0 0) (end 2.75 0) (layer Cmts.User) (width 0.15))
+    (fp_circle (center 0 0) (end 3 0) (layer F.CrtYd) (width 0.05))
+    (pad 1 thru_hole circle (at 0 0) (size 5.5 5.5) (drill 3.2) (layers *.Cu *.Mask))
+  )
+  (module Mounting_Holes:MountingHole_3.2mm_M3_ISO14580_Pad (layer F.Cu)
+    (at 60 132.5)
+    (descr "Mounting Hole 3.2mm, M3, ISO14580")
+    (tags "mounting hole 3.2mm m3 iso14580")
+    (fp_text reference REF** (at 0 -3.75) (layer F.SilkS)
+      (effects (font (size 1 1) (thickness 0.15)))
+    )
+    (fp_text value MountingHole_3.2mm_M3_ISO14580_Pad (at 0 3.75) (layer F.Fab)
+      (effects (font (size 1 1) (thickness 0.15)))
+    )
+    (fp_circle (center 0 0) (end 2.75 0) (layer Cmts.User) (width 0.15))
+    (fp_circle (center 0 0) (end 3 0) (layer F.CrtYd) (width 0.05))
+    (pad 1 thru_hole circle (at 0 0) (size 5.5 5.5) (drill 3.2) (layers *.Cu *.Mask))
+  )
+  (module Mounting_Holes:MountingHole_3.2mm_M3_ISO14580_Pad (layer F.Cu)
+    (at 140 132.5)
+    (descr "Mounting Hole 3.2mm, M3, ISO14580")
+    (tags "mounting hole 3.2mm m3 iso14580")
+    (fp_text reference REF** (at 0 -3.75) (layer F.SilkS)
+      (effects (font (size 1 1) (thickness 0.15)))
+    )
+    (fp_text value MountingHole_3.2mm_M3_ISO14580_Pad (at 0 3.75) (layer F.Fab)
+      (effects (font (size 1 1) (thickness 0.15)))
+    )
+    (fp_circle (center 0 0) (end 2.75 0) (layer Cmts.User) (width 0.15))
+    (fp_circle (center 0 0) (end 3 0) (layer F.CrtYd) (width 0.05))
+    (pad 1 thru_hole circle (at 0 0) (size 5.5 5.5) (drill 3.2) (layers *.Cu *.Mask))
+  )
+  (gr_text V1.0 (at 125.984 122.2248) (layer F.SilkS)
+    (effects (font (size 3 3) (thickness 0.3)))
+  )
+  (gr_text MoonStalker (at 126.492 117.9576) (layer F.SilkS)
+    (effects (font (size 3 3) (thickness 0.3)))
+  )
   (gr_line (start 146.05 53.34) (end 54.61 53.34) (angle 90) (layer Edge.Cuts) (width 0.15))
